File: c128-sram.kicad_pcb (KiCad board)
At the start: 2 copper layers, 30.2 x 35.6 mm, 17 parts, among them J1 Jumper, J2 Jumper, J3 Jumper, J4 Jumper, U1 74AHCT32, U2 74AHCT573, U3 IS61C1024AL-32TSOP, U4 74AHCT1G00, U49 DRAM-4164, U50 DRAM-4164

Commit message: Add files via upload
Parts:
- U4: value 74AHCT1G00 -> 74AHCT2G00DC,125; footprint Package_SO:TSOP-5_1.65x3.05mm_P0.95mm -> Package_SO:VSSOP-8_2.4x2.1mm_P0.5mm
- moved U4 1.49 mm to (68.5, 106.2), turned to 270 degrees
- renumbered RIGHT3 to X1, LEFT3 to X2, /RC1 to X3
Connections:
- U3 pad 6: Net-(U1-Pad10) -> Net-(U3-Pad6)
- U4 pad 3: GND -> Net-(U1-Pad10)
- U4 pad 4: Net-(U1-Pad10) -> GND
- U4 pad 5: +5V -> Net-(U3-Pad6)
Routing:
- net Net-(U3-Pad6): track 0.00 -> 6.68 mm, vias 0 -> 1
- net Net-(U1-Pad10): track 28.4 -> 24.0 mm, vias 3 -> 2
- net Net-(U4-Pad2): track 10.5 -> 12.6 mm
- net Net-(U3-Pad10): track 16.4 -> 18.5 mm
- net +5V: track 80.4 -> 79.3 mm, vias 1 -> 2
- net GND: track 92.4 -> 91.6 mm
